File: kicad-files/rev1/patch-shield.sch (KiCad schematic (older format))
At the start: 18 parts

Commit message: added connectors for lead-wire shields
Parts:
- added P? (x16): CONN_1, symbol CONN_1
Connections:
- wire segments 49 -> 81

Commit message: move LEDs to patch-shield
Parts:
- added D? (x32): LED, symbol LED
- added R? (x16): 560, symbol R
Connections:
- net labels added: DGND, GREEN_1N, GREEN_1P, GREEN_2N, GREEN_2P, GREEN_3N, GREEN_3P, GREEN_4N, GREEN_4P, GREEN_5N, GREEN_5P, GREEN_6N, GREEN_6P, GREEN_7N, GREEN_7P, GREEN_8N, GREEN_8P, YELLOW_1N, YELLOW_1P, YELLOW_2N, YELLOW_2P, YELLOW_3N, YELLOW_3P, YELLOW_4N, YELLOW_4P, YELLOW_5N, YELLOW_5P, YELLOW_6N, YELLOW_6P, YELLOW_7N, YELLOW_7P, YELLOW_8N, YELLOW_8P
- wire segments 81 -> 179

Commit message: added shift-out register for LEDs
Parts:
- added P?: CONN_4X2, symbol CONN_4X2
- added U? (x4): 74HC595, symbol 74HC595
Connections:
- net labels added: +3.3V, LED_LATCH_CLK, LED_OUTPUT_ENABLE_INPUT, LED_SERIAL, LED_SHIFT_REG_CLEAR, LED_SHIFT_REG_CLK
- wire segments 179 -> 263
Other:
- moved on the sheet: P?

Commit message: added power LED for patch shield
Parts:
- added D?: LED, symbol LED
- added R?: 560, symbol R
Connections:
- wire segments 263 -> 268
Other:
- note added: "Power Indicator"
Changed lines of the file:
@@
-EESchema Schematic File Version 2  date Sat 25 May 2013 05:38:00 PM CEST
+EESchema Schematic File Version 2  date Sat 25 May 2013 06:06:03 PM CEST
 LIBS:power
 LIBS:device
@@
 Comment4 ""
 $EndDescr
+Text Notes 5300 6500 0    60   ~ 0
+Power Indicator
+Wire Wire Line
+	6650 6800 6650 6600
+Wire Wire Line
+	5200 6600 5000 6600
+Wire Wire Line
+	6000 6600 5700 6600
 Connection ~ 6300 6000
 Wire Wire Line
@@
 Connection ~ 5250 1250
 Wire Wire Line
-	5750 3750 5750 3400
+	5750 3400 5750 3750
 Wire Wire Line
 	5350 3100 3850 3100
@@
 	5050 5200 5300 5200
 Connection ~ 5300 5200
+Wire Wire Line
+	6650 6600 6400 6600
+Wire Wire Line
+	5000 6600 5000 6450
+$Comp
+L DGND #PWR?
+U 1 1 51A0E103
+P 6650 6800
+F 0 "#PWR?" H 6650 6800 40  0001 C CNN
+F 1 "DGND" H 6650 6730 40  0000 C CNN
+	1    6650 6800
+	1    0    0    -1
+$EndComp
+$Comp
+L +3.3V #PWR?
+U 1 1 51A0E0F7
+P 5000 6450
+F 0 "#PWR?" H 5000 6410 30  0001 C CNN
+F 1 "+3.3V" H 5000 6560 30  0000 C CNN
+	1    5000 6450
+	1    0    0    -1
+$EndComp
+$Comp
+L R R?
+U 1 1 51A0E0BF
+P 5450 6600
+F 0 "R?" V 5530 6600 50  0000 C CNN
+F 1 "560" V 5450 6600 50  0000 C CNN
+	1    5450 6600
+	0    -1   1    0
+$EndComp
+$Comp
+L LED D?
+U 1 1 51A0E0BE
+P 6200 6600
+F 0 "D?" H 6200 6700 50  0000 C CNN
+F 1 "LED" H 6200 6500 50  0000 C CNN
+	1    6200 6600
+	1    0    0    1
+$EndComp
 $Comp
 L PWR_FLAG #FLG?

Commit message: Added decoupling caps and ferrite to patch shield
Parts:
- added C? (x4): 10uF, symbol C
- added C? (x4): 100nF, symbol C
- added L?: INDUCTOR, symbol INDUCTOR
Connections:
- wire segments 268 -> 292

Commit message: Patch shield schematic cleanup
Connections:
- wire segments 292 -> 294
Other:
- moved on the sheet: C?

Commit message: move RS-485 to the patch-shield
Parts:
- removed P?: CONN_4X2, symbol CONN_4X2
- added C? (x4): 100nF, symbol C
- added C?: 10uF, symbol C
- added D? (x4): DOUBLE_SCHOTTKY, symbol DOUBLE_SCHOTTKY
- added J? (x2): RJ45, symbol RJ45
- added L?: INDUCTOR, symbol INDUCTOR
- added P?: CONN_8X2, symbol CONN_8X2
- added P?: ARDUINO_SHIELD, symbol ARDUINO_SHIELD
- added R? (x2): 680, symbol R
- added R?: 120, symbol R
- added R? (x6): 1k, symbol R
- added R? (x3): 100k, symbol R
- added U?: 74HC00, symbol 7400
- added U? (x2): TS5A4624, symbol TS5A4624
- added U?: RS485, symbol RS485
Connections:
- net labels added: +5V, 5V_IN, DAISY_DETECT_NEXT, DAISY_DETECT_NEXT_FILT, DAISY_DETECT_PREVIOUS, DAISY_DETECT_PREVIOUS_FILT, DAISY_ENUMERATION_IN, DAISY_ENUMERATION_IN_FILT, DAISY_ENUMERATION_OUT, DAISY_ENUMERATION_OUT_FILT, GND, PA16, PA17, PA18, PA22, PA23, PA24, PA25, PA26, PA27, PA28, PA29, PA4, PA6, PA8, PA9, PB25, PB27, PC21, PC22, PC23, PC24, PC25, PC26, PC28, PC29, PD7, PD8, RESET, RS485_A, RS485_B, RTS2_RS485_DE, RXD2_RS485_R, TXD2_RS485_D, V_IN
- net labels removed: DGND
- wire segments 294 -> 456
- no-connect marks 0 -> 3
Other:
- note added: "Biasing and termination for RS-485"
- note added: "DAISY CHAIN NEXT"
- note added: "DAISY CHAIN PREVIOUS"
- note added: "TODO: Replace with SN74LVC1G00DCKR"
- note added: "TODO: according to the SN65HVD78D datasheet, \n we may not need the biasing resistors \n (allowing us to eleminate a switch). \n We should discuss this."
- note added: "e.g. SN65HVD78D"
- moved on the sheet: C?, D?, L?, P?, R?
