File: kicad-files/rev1/patch-shield-analog.sch (KiCad schematic (older format))
At the start: 38 parts

Commit message: bring ADS129x_GPIO headers up to the digital shield
Parts:
- added P?: CONN_4, symbol CONN_4
Connections:
- net labels added: ADS129x_GPIO1, ADS129x_GPIO2, ADS129x_GPIO3, ADS129x_GPIO4
- wire segments 204 -> 208
Changed lines of the file:
@@
-EESchema Schematic File Version 2  date Sat 08 Jun 2013 07:26:01 PM CEST
+EESchema Schematic File Version 2  date Sun 09 Jun 2013 09:26:44 AM CEST
 LIBS:power
 LIBS:device
@@
 LIBS:analog-switches
 LIBS:arduino-shield
+LIBS:patch-shield-analog-cache
 EELAYER 25  0
 EELAYER END
@@
 Sheet 1 1
 Title "noname.sch"
-Date "8 jun 2013"
+Date "9 jun 2013"
 Rev ""
 Comp ""
@@
 $EndDescr
 $Comp
+L CONN_4 P?
+U 1 1 51B42E2E
+P 7250 1000
+F 0 "P?" V 7200 1000 50  0000 C CNN
+F 1 "CONN_4" V 7300 1000 50  0000 C CNN
+	1    7250 1000
+	1    0    0    -1
+$EndComp
+Text Label 5300 1150 0    60   ~ 0
+ADS129x_GPIO4
+Text Label 5300 1050 0    60   ~ 0
+ADS129x_GPIO3
+Text Label 5300 950  0    60   ~ 0
+ADS129x_GPIO2
+Text Label 5300 850  0    60   ~ 0
+ADS129x_GPIO1
+Wire Wire Line
+	5300 850  6900 850
+Wire Wire Line
+	5300 950  6900 950
+Wire Wire Line
+	5300 1050 6900 1050
+Wire Wire Line
+	5300 1150 6900 1150
+$Comp
 L AGND #PWR?

Commit message: improve text label names
Connections:
- net labels added: PA16_A0, PA17_SDA1, PA18_SCL1, PA22_A3, PA23_A2, PA24_A1, PA25_MISO, PA26_MOSI, PA27_SCLK, PA28_SS0, PA29_SS1, PA4_A5, PA6_A4, PA8_RX, PA9_TX, PB25_PWM2, PB27_PWM13, PC21_PWM9, PC22_PWM8, PC23_PWM7, PC24_PWM6, PC25_PWM5, PC26_PWM4, PC28_PWM3, PC29_PWM10, PD7_PWM11, PD8_PWM12
- net labels removed: PA16, PA17, PA18, PA22, PA23, PA24, PA25, PA26, PA27, PA28, PA29, PA4, PA6, PA8, PA9, PB25, PB27, PC21, PC22, PC23, PC24, PC25, PC26, PC28, PC29, PD7, PD8
Changed lines of the file:
@@
 $EndComp
 Text Label 6450 2900 0    60   ~ 0
-PA16
+PA16_A0
 Text Label 6450 3000 0    60   ~ 0
-PA24
+PA24_A1
 Text Label 6450 3100 0    60   ~ 0
-PA23
+PA23_A2
 Text Label 6450 3200 0    60   ~ 0
-PA22
+PA22_A3
 Text Label 6450 3300 0    60   ~ 0
-PA6
+PA6_A4
 Text Label 6450 3400 0    60   ~ 0
-PA4
+PA4_A5
 Text Label 10550 3400 2    60   ~ 0
-PA8
+PA8_RX
 Text Label 10550 3300 2    60   ~ 0
-PA9
+PA9_TX
 Text Label 10550 3200 2    60   ~ 0
-PB25
+PB25_PWM2
 Text Label 10550 3100 2    60   ~ 0
-PC28
+PC28_PWM3
 Text Label 11050 3000 2    60   ~ 0
-PA29
+PA29_SS1
 Text Label 11050 2900 2    60   ~ 0
-PC26
+PC26_PWM4
 Text Label 10550 2900 2    60   ~ 0
-PC25
+PC25_PWM5
 Text Label 10550 2800 2    60   ~ 0
-PC24
+PC24_PWM6
 Text Label 10550 2700 2    60   ~ 0
-PC23
+PC23_PWM7
 Text Label 10550 2500 2    60   ~ 0
-PC22
+PC22_PWM8
 Text Label 10550 2400 2    60   ~ 0
-PC21
+PC21_PWM9
 Text Label 11050 2300 2    60   ~ 0
-PA28
+PA28_SS0
 Text Label 11050 2200 2    60   ~ 0
-PC29
+PC29_PWM10
 Text Label 10550 2200 2    60   ~ 0
-PD7
+PD7_PWM11
 Text Label 10550 2100 2    60   ~ 0
-PD8
+PD8_PWM12
 Text Label 10550 2000 2    60   ~ 0
-PB27
+PB27_PWM13
 $Comp
 L GND #PWR?
@@
 $EndComp
 Text Label 10550 1700 2    60   ~ 0
-PA17
+PA17_SDA1
 Text Label 10550 1600 2    60   ~ 0
-PA18
+PA18_SCL1
 NoConn ~ 10550 1800
 $Comp
@@
 $EndComp
 Text Label 9950 4050 2    60   ~ 0
-PA26
+PA26_MOSI
 Text Label 6950 3950 0    60   ~ 0
-PA25
+PA25_MISO
 Text Label 6950 4050 0    60   ~ 0
-PA27
+PA27_SCLK
 Text Label 6950 4150 0    60   ~ 0
 RESET

Commit message: tidy up the labels and wires on the shields
Other:
- moved on the sheet: P?

Commit message: Fixed patch shield to pass ERC
Parts:
- gave numbers to parts that had none: 39
Connections:
- net labels removed: +3.3V, +5V, ADS129x_GPIO1, ADS129x_GPIO2, ADS129x_GPIO3, ADS129x_GPIO4, DAISY_DETECT_NEXT_FILT, DAISY_DETECT_PREVIOUS_FILT, DAISY_ENUMERATION_IN_FILT, DAISY_ENUMERATION_OUT_FILT, GND, LED_LATCH_CLK, LED_OUTPUT_ENABLE_INPUT, LED_SERIAL, LED_SHIFT_REG_CLEAR, LED_SHIFT_REG_CLK, PA16_A0, PA17_SDA1, PA18_SCL1, PA22_A3, PA23_A2, PA24_A1, PA25_MISO, PA26_MOSI, PA27_SCLK, PA28_SS0, PA29_SS1, PA4_A5, PA6_A4, PA8_RX, PA9_TX, PB25_PWM2, PB27_PWM13, PC21_PWM9, PC22_PWM8, PC23_PWM7, PC24_PWM6, PC25_PWM5, PC26_PWM4, PC28_PWM3, PC29_PWM10, PD7_PWM11, PD8_PWM12, RESET, RTS2_RS485_DE, RXD2_RS485_R, TXD2_RS485_D, V_IN
- wire segments 208 -> 86
- no-connect marks 1 -> 58
Other:
- moved on the sheet: P35

Commit message: remove RS-485
 The purpose of the RS-485 was to allow us to synch multiple
devices. However, a better way to do this is to inject a counter
into the samples using the USB Start Of Frame which will be
shared by all devices on the same USB bus.
Parts:
- removed P37: CONN_8X2, symbol CONN_8X2
- added P37: CONN_4X2, symbol CONN_4X2
Connections:
- no-connect marks 58 -> 50
Changed lines of the file:
@@
-EESchema Schematic File Version 2  date Fri 21 Jun 2013 09:55:02 PM UTC
+EESchema Schematic File Version 2  date Sat 22 Jun 2013 01:13:28 PM CEST
 LIBS:power
 LIBS:device
@@
 LIBS:analog-switches
 LIBS:arduino-shield
+LIBS:patch-shield-analog-cache
 EELAYER 25  0
 EELAYER END
@@
 Sheet 1 1
 Title "noname.sch"
-Date "21 jun 2013"
+Date "22 jun 2013"
 Rev ""
 Comp ""
@@
 Comment4 ""
 $EndDescr
+$Comp
+L CONN_4X2 P37
+U 1 1 51C586AC
+P 7800 5450
+F 0 "P37" H 7800 5700 50  0000 C CNN
+F 1 "CONN_4X2" V 7800 5450 40  0000 C CNN
+	1    7800 5450
+	1    0    0    -1
+$EndComp
 NoConn ~ 7400 5300
-NoConn ~ 7400 5700
 NoConn ~ 8200 5500
 NoConn ~ 8700 4150
@@
 NoConn ~ 9000 1700
 NoConn ~ 9000 1600
-NoConn ~ 8200 6000
-NoConn ~ 8200 5900
-NoConn ~ 8200 5800
-NoConn ~ 8200 5700
 NoConn ~ 8200 5600
 NoConn ~ 8200 5400
@@
 NoConn ~ 7400 5500
 NoConn ~ 7400 5600
-NoConn ~ 7400 5800
-NoConn ~ 7400 5900
-NoConn ~ 7400 6000
 NoConn ~ 6900 1150
 NoConn ~ 6900 1050
@@
 $EndComp
 $Comp
-L AGND #PWR01
+L AGND #PWR4
 U 1 1 51B368C7
 P 3600 1350
-F 0 "#PWR01" H 3600 1350 40  0001 C CNN
+F 0 "#PWR4" H 3600 1350 40  0001 C CNN
 F 1 "AGND" H 3600 1280 50  0000 C CNN
 	1    3600 1350
@@
 	3600 1350 3600 1150
 $Comp
-L +5VA #PWR02
+L +5VA #PWR1
 U 1 1 51B368B6
 P 1950 900
-F 0 "#PWR02" H 1950 1030 20  0001 C CNN
+F 0 "#PWR1" H 1950 1030 20  0001 C CNN
 F 1 "+5VA" H 1950 1000 30  0000 C CNN
 	1    1950 900
@@
 F 1 "ARDUINO_SHIELD" H 7700 2600 60  0000 C CNN
 	1    7700 2600
-	1    0    0    -1
-$EndComp
-$Comp
-L CONN_8X2 P37
-U 1 1 51B34A08
-P 7800 5650
-F 0 "P37" H 7800 6100 60  0000 C CNN
-F 1 "CONN_8X2" V 7800 5650 50  0000 C CNN
-	1    7800 5650
 	1    0    0    -1
 $EndComp
@@
 $EndComp
 $Comp
-L PWR_FLAG #FLG03
+L PWR_FLAG #FLG2
 U 1 1 51A0AF7D
 P 2600 4100
-F 0 "#FLG03" H 2600 4195 30  0001 C CNN
+F 0 "#FLG2" H 2600 4195 30  0001 C CNN
 F 1 "PWR_FLAG" H 2600 4280 30  0000 C CNN
 	1    2600 4100
@@
 $EndComp
 $Comp
-L PWR_FLAG #FLG04
+L PWR_FLAG #FLG1
 U 1 1 51A0AF32
 P 2150 1600
-F 0 "#FLG04" H 2150 1695 30  0001 C CNN
+F 0 "#FLG1" H 2150 1695 30  0001 C CNN
 F 1 "PWR_FLAG" H 2150 1780 30  0000 C CNN
 	1    2150 1600
@@
 $EndComp
 $Comp
-L +5VA #PWR05
+L +5VA #PWR2
 U 1 1 51A0AEED
 P 2400 1500
-F 0 "#PWR05" H 2400 1630 20  0001 C CNN
+F 0 "#PWR2" H 2400 1630 20  0001 C CNN
 F 1 "+5VA" H 2400 1600 30  0000 C CNN
 	1    2400 1500
@@
 $EndComp
 $Comp
-L AGND #PWR06
+L AGND #PWR3
 U 1 1 51A0AD37
 P 2900 4200
-F 0 "#PWR06" H 2900 4200 40  0001 C CNN
+F 0 "#PWR3" H 2900 4200 40  0001 C CNN
 F 1 "AGND" H 2900 4130 50  0000 C CNN
 	1    2900 4200

Commit message: starting analog patch shield layout
Parts:
- D1, R1: footprint (none) -> SM0603
- P1, P10, P11, P12, P13, P14, P15, P16, P17, P19, P2, P20, P21, P22, P23, P24, P25, P26, P27, P28, P29, P3, P30, P31, P32, P33, P34, P4, P5, P6, P7, P8, P9: footprint (none) -> Touchproof-socket
- P18: footprint (none) -> PIN_ARRAY_20X2
- P35: footprint (none) -> PIN_ARRAY_4x1
- P36: footprint (none) -> arduino_shield
- P37: footprint (none) -> pin_array_4x2
Changed lines of the file:
@@
-EESchema Schematic File Version 2  date Sat 22 Jun 2013 01:13:28 PM CEST
+EESchema Schematic File Version 2  date Sat 22 Jun 2013 05:02:41 PM CEST
 LIBS:power
 LIBS:device
@@
 F 0 "P37" H 7800 5700 50  0000 C CNN
 F 1 "CONN_4X2" V 7800 5450 40  0000 C CNN
+F 2 "pin_array_4x2" V 7900 5450 40  0001 C CNN
 	1    7800 5450
 	1    0    0    -1
@@
 F 0 "P35" V 7200 1000 50  0000 C CNN
 F 1 "CONN_4" V 7300 1000 50  0000 C CNN
+F 2 "PIN_ARRAY_4x1" V 7400 1000 50  0001 C CNN
 	1    7250 1000
 	1    0    0    -1
 $EndComp
 $Comp
-L AGND #PWR4
+L AGND #PWR01
 U 1 1 51B368C7
 P 3600 1350
-F 0 "#PWR4" H 3600 1350 40  0001 C CNN
+F 0 "#PWR01" H 3600 1350 40  0001 C CNN
 F 1 "AGND" H 3600 1280 50  0000 C CNN
 	1    3600 1350
@@
 	3600 1350 3600 1150
 $Comp
-L +5VA #PWR1
+L +5VA #PWR02
 U 1 1 51B368B6
 P 1950 900
-F 0 "#PWR1" H 1950 1030 20  0001 C CNN
+F 0 "#PWR02" H 1950 1030 20  0001 C CNN
 F 1 "+5VA" H 1950 1000 30  0000 C CNN
 	1    1950 900
@@
 F 0 "P36" H 7700 2800 60  0000 C CNN
 F 1 "ARDUINO_SHIELD" H 7700 2600 60  0000 C CNN
+F 2 "arduino_shield" H 7700 2700 60  0001 C CNN
 	1    7700 2600
 	1    0    0    -1
@@
 F 0 "R1" V 2480 1150 50  0000 C CNN
 F 1 "1k" V 2400 1150 50  0000 C CNN
+F 2 "SM0603" V 2500 1150 50  0001 C CNN
 	1    2400 1150
 	0    -1   1    0
@@
 F 0 "D1" H 3150 1250 50  0000 C CNN
 F 1 "LED" H 3150 1050 50  0000 C CNN
+F 2 "SM0603" H 3150 1150 50  0001 C CNN
 	1    3150 1150
 	1    0    0    1
@@
 F 0 "P2" H 1280 1950 40  0000 L CNN
 F 1 "CONN_1" H 1200 2005 30  0001 C CNN
+F 2 "Touchproof-socket" H 1200 2105 30  0001 C CNN
 	1    1200 1950
 	-1   0    0    -1
@@
 F 0 "P3" H 1280 2150 40  0000 L CNN
 F 1 "CONN_1" H 1200 2205 30  0001 C CNN
+F 2 "Touchproof-socket" H 1200 2305 30  0001 C CNN
 	1    1200 2150
 	-1   0    0    -1
@@
 F 0 "P5" H 1280 2550 40  0000 L CNN
 F 1 "CONN_1" H 1200 2605 30  0001 C CNN
+F 2 "Touchproof-socket" H 1200 2705 30  0001 C CNN
 	1    1200 2550
 	-1   0    0    -1
@@
 F 0 "P4" H 1280 2350 40  0000 L CNN
 F 1 "CONN_1" H 1200 2405 30  0001 C CNN
+F 2 "Touchproof-socket" H 1200 2505 30  0001 C CNN
 	1    1200 2350
 	-1   0    0    -1
@@
 F 0 "P8" H 1280 3150 40  0000 L CNN
 F 1 "CONN_1" H 1200 3205 30  0001 C CNN
+F 2 "Touchproof-socket" H 1200 3305 30  0001 C CNN
 	1    1200 3150
 	-1   0    0    -1
@@
 F 0 "P9" H 1280 3350 40  0000 L CNN
 F 1 "CONN_1" H 1200 3405 30  0001 C CNN
+F 2 "Touchproof-socket" H 1200 3505 30  0001 C CNN
 	1    1200 3350
 	-1   0    0    -1
@@
 F 0 "P7" H 1280 2950 40  0000 L CNN
 F 1 "CONN_1" H 1200 3005 30  0001 C CNN
+F 2 "Touchproof-socket" H 1200 3105 30  0001 C CNN
 	1    1200 2950
 	-1   0    0    -1
@@
 F 0 "P6" H 1280 2750 40  0000 L CNN
 F 1 "CONN_1" H 1200 2805 30  0001 C CNN
+F 2 "Touchproof-socket" H 1200 2905 30  0001 C CNN
 	1    1200 2750
 	-1   0    0    -1
@@
 F 0 "P31" H 4680 2750 40  0000 L CNN
 F 1 "CONN_1" H 4600 2805 30  0001 C CNN
+F 2 "Touchproof-socket" H 4600 2905 30  0001 C CNN
 	1    4600 2750
 	1    0    0    -1
@@
 F 0 "P32" H 4680 2950 40  0000 L CNN
 F 1 "CONN_1" H 4600 3005 30  0001 C CNN
+F 2 "Touchproof-socket" H 4600 3105 30  0001 C CNN
 	1    4600 2950
 	1    0    0    -1
@@
 F 0 "P34" H 4680 3350 40  0000 L CNN
 F 1 "CONN_1" H 4600 3405 30  0001 C CNN
+F 2 "Touchproof-socket" H 4600 3505 30  0001 C CNN
 	1    4600 3350
 	1    0    0    -1
@@
 F 0 "P33" H 4680 3150 40  0000 L CNN
 F 1 "CONN_1" H 4600 3205 30  0001 C CNN
+F 2 "Touchproof-socket" H 4600 3305 30  0001 C CNN
 	1    4600 3150
 	1    0    0    -1
@@
 F 0 "P29" H 4680 2350 40  0000 L CNN
 F 1 "CONN_1" H 4600 2405 30  0001 C CNN
+F 2 "Touchproof-socket" H 4600 2505 30  0001 C CNN
 	1    4600 2350
 	1    0    0    -1
@@
 F 0 "P30" H 4680 2550 40  0000 L CNN
 F 1 "CONN_1" H 4600 2605 30  0001 C CNN
+F 2 "Touchproof-socket" H 4600 2705 30  0001 C CNN
 	1    4600 2550
 	1    0    0    -1
@@
 F 0 "P28" H 4680 2150 40  0000 L CNN
 F 1 "CONN_1" H 4600 2205 30  0001 C CNN
+F 2 "Touchproof-socket" H 4600 2305 30  0001 C CNN
 	1    4600 2150
 	1    0    0    -1
@@
 F 0 "P27" H 4680 1950 40  0000 L CNN
 F 1 "CONN_1" H 4600 2005 30  0001 C CNN
+F 2 "Touchproof-socket" H 4600 2105 30  0001 C CNN
 	1    4600 1950
 	1    0    0    -1
@@
 F 0 "P1" H 930 3550 40  0000 L CNN
 F 1 "CONN_1" H 850 3605 30  0001 C CNN
+F 2 "Touchproof-socket" H 850 3705 30  0001 C CNN
 	1    850  3550
 	-1   0    0    -1
 $EndComp
 $Comp
-L PWR_FLAG #FLG2
+L PWR_FLAG #FLG03
 U 1 1 51A0AF7D
 P 2600 4100
-F 0 "#FLG2" H 2600 4195 30  0001 C CNN
+F 0 "#FLG03" H 2600 4195 30  0001 C CNN
 F 1 "PWR_FLAG" H 2600 4280 30  0000 C CNN
 	1    2600 4100
@@
 $EndComp
 $Comp
-L PWR_FLAG #FLG1
+L PWR_FLAG #FLG04
 U 1 1 51A0AF32
 P 2150 1600
-F 0 "#FLG1" H 2150 1695 30  0001 C CNN
+F 0 "#FLG04" H 2150 1695 30  0001 C CNN
 F 1 "PWR_FLAG" H 2150 1780 30  0000 C CNN
 	1    2150 1600
@@
 $EndComp
 $Comp
-L +5VA #PWR2
+L +5VA #PWR05
 U 1 1 51A0AEED
 P 2400 1500
-F 0 "#PWR2" H 2400 1630 20  0001 C CNN
+F 0 "#PWR05" H 2400 1630 20  0001 C CNN
 F 1 "+5VA" H 2400 1600 30  0000 C CNN
 	1    2400 1500
@@
 F 0 "P10" H 1680 1950 40  0000 L CNN
 F 1 "CONN_1" H 1600 2005 30  0001 C CNN
+F 2 "Touchproof-socket" H 1600 2105 30  0001 C CNN
 	1    1600 1950
 	-1   0    0    -1
@@
 F 0 "P11" H 1680 2150 40  0000 L CNN
 F 1 "CONN_1" H 1600 2205 30  0001 C CNN
+F 2 "Touchproof-socket" H 1600 2305 30  0001 C CNN
 	1    1600 2150
 	-1   0    0    -1
@@
 F 0 "P13" H 1680 2550 40  0000 L CNN
 F 1 "CONN_1" H 1600 2605 30  0001 C CNN
+F 2 "Touchproof-socket" H 1600 2705 30  0001 C CNN
 	1    1600 2550
 	-1   0    0    -1
@@
 F 0 "P12" H 1680 2350 40  0000 L CNN
 F 1 "CONN_1" H 1600 2405 30  0001 C CNN
+F 2 "Touchproof-socket" H 1600 2505 30  0001 C CNN
 	1    1600 2350
 	-1   0    0    -1
@@
 F 0 "P16" H 1680 3150 40  0000 L CNN
 F 1 "CONN_1" H 1600 3205 30  0001 C CNN
+F 2 "Touchproof-socket" H 1600 3305 30  0001 C CNN
 	1    1600 3150
 	-1   0    0    -1
@@
 F 0 "P17" H 1680 3350 40  0000 L CNN
 F 1 "CONN_1" H 1600 3405 30  0001 C CNN
+F 2 "Touchproof-socket" H 1600 3505 30  0001 C CNN
 	1    1600 3350
 	-1   0    0    -1
@@
 F 0 "P15" H 1680 2950 40  0000 L CNN
 F 1 "CONN_1" H 1600 3005 30  0001 C CNN
+F 2 "Touchproof-socket" H 1600 3105 30  0001 C CNN
 	1    1600 2950
 	-1   0    0    -1
@@
 F 0 "P14" H 1680 2750 40  0000 L CNN
 F 1 "CONN_1" H 1600 2805 30  0001 C CNN
+F 2 "Touchproof-socket" H 1600 2905 30  0001 C CNN
 	1    1600 2750
 	-1   0    0    -1
 $EndComp
 $Comp
-L AGND #PWR3
+L AGND #PWR06
 U 1 1 51A0AD37
 P 2900 4200
-F 0 "#PWR3" H 2900 4200 40  0001 C CNN
+F 0 "#PWR06" H 2900 4200 40  0001 C CNN
 F 1 "AGND" H 2900 4130 50  0000 C CNN
 	1    2900 4200
@@
 F 0 "P23" H 4280 2750 40  0000 L CNN
 F 1 "CONN_1" H 4200 2805 30  0001 C CNN
+F 2 "Touchproof-socket" H 4200 2905 30  0001 C CNN
 	1    4200 2750
 	1    0    0    -1
@@
 F 0 "P24" H 4280 2950 40  0000 L CNN
 F 1 "CONN_1" H 4200 3005 30  0001 C CNN
+F 2 "Touchproof-socket" H 4200 3105 30  0001 C CNN
 	1    4200 2950
 	1    0    0    -1
@@
 F 0 "P26" H 4280 3350 40  0000 L CNN
 F 1 "CONN_1" H 4200 3405 30  0001 C CNN
+F 2 "Touchproof-socket" H 4200 3505 30  0001 C CNN
 	1    4200 3350
 	1    0    0    -1
@@
 F 0 "P25" H 4280 3150 40  0000 L CNN
 F 1 "CONN_1" H 4200 3205 30  0001 C CNN
+F 2 "Touchproof-socket" H 4200 3305 30  0001 C CNN
 	1    4200 3150
 	1    0    0    -1
@@
 F 0 "P21" H 4280 2350 40  0000 L CNN
 F 1 "CONN_1" H 4200 2405 30  0001 C CNN
+F 2 "Touchproof-socket" H 4200 2505 30  0001 C CNN
 	1    4200 2350
 	1    0    0    -1
@@
 F 0 "P22" H 4280 2550 40  0000 L CNN
 F 1 "CONN_1" H 4200 2605 30  0001 C CNN
+F 2 "Touchproof-socket" H 4200 2705 30  0001 C CNN
 	1    4200 2550
 	1    0    0    -1
@@
 F 0 "P20" H 4280 2150 40  0000 L CNN
 F 1 "CONN_1" H 4200 2205 30  0001 C CNN
+F 2 "Touchproof-socket" H 4200 2305 30  0001 C CNN
 	1    4200 2150
 	1    0    0    -1
@@
 F 0 "P19" H 4280 1950 40  0000 L CNN
 F 1 "CONN_1" H 4200 2005 30  0001 C CNN
+F 2 "Touchproof-socket" H 4200 2105 30  0001 C CNN
 	1    4200 1950
 	1    0    0    -1
@@
 F 0 "P18" H 2900 3750 60  0000 C CNN
 F 1 "CONN_20X2" V 2900 2700 50  0000 C CNN
+F 2 "PIN_ARRAY_20X2" V 3000 2700 50  0001 C CNN
 	1    2900 2700
 	1    0    0    -1

Commit message: merge GPIO and Supplemental IO connectors
Parts:
- removed P35: CONN_4, PIN_ARRAY_4x1, symbol CONN_4
- removed P37: CONN_4X2, pin_array_4x2, symbol CONN_4X2
- added P35: CONN_5X2, symbol CONN_5X2
Connections:
- no-connect marks 50 -> 47
Changed lines of the file:
@@
-EESchema Schematic File Version 2  date Sat 22 Jun 2013 05:02:41 PM CEST
+EESchema Schematic File Version 2  date Sat 06 Jul 2013 02:58:34 PM CEST
 LIBS:power
 LIBS:device
@@
 Sheet 1 1
 Title "noname.sch"
-Date "22 jun 2013"
+Date "6 jul 2013"
 Rev ""
 Comp ""
@@
 Comment4 ""
 $EndDescr
-$Comp
-L CONN_4X2 P37
-U 1 1 51C586AC
-P 7800 5450
-F 0 "P37" H 7800 5700 50  0000 C CNN
-F 1 "CONN_4X2" V 7800 5450 40  0000 C CNN
-F 2 "pin_array_4x2" V 7900 5450 40  0001 C CNN
-	1    7800 5450
+NoConn ~ 8200 5700
+NoConn ~ 7400 5700
+$Comp
+L CONN_5X2 P35
+U 1 1 51D81450
+P 7800 5500
+F 0 "P35" H 7800 5800 60  0000 C CNN
+F 1 "CONN_5X2" V 7800 5500 50  0000 C CNN
+	1    7800 5500
 	1    0    0    -1
 $EndComp
@@
 NoConn ~ 7400 5500
 NoConn ~ 7400 5600
-NoConn ~ 6900 1150
-NoConn ~ 6900 1050
-NoConn ~ 6900 950
-NoConn ~ 6900 850
-NoConn ~ 6900 850
-$Comp
-L CONN_4 P35
-U 1 1 51B42E2E
-P 7250 1000
-F 0 "P35" V 7200 1000 50  0000 C CNN
-F 1 "CONN_4" V 7300 1000 50  0000 C CNN
-F 2 "PIN_ARRAY_4x1" V 7400 1000 50  0001 C CNN
-	1    7250 1000
-	1    0    0    -1
-$EndComp
-$Comp
-L AGND #PWR01
+$Comp
+L AGND #PWR4
 U 1 1 51B368C7
 P 3600 1350
-F 0 "#PWR01" H 3600 1350 40  0001 C CNN
+F 0 "#PWR4" H 3600 1350 40  0001 C CNN
 F 1 "AGND" H 3600 1280 50  0000 C CNN
 	1    3600 1350
@@
 	3600 1350 3600 1150
 $Comp
-L +5VA #PWR02
+L +5VA #PWR1
 U 1 1 51B368B6
 P 1950 900
-F 0 "#PWR02" H 1950 1030 20  0001 C CNN
+F 0 "#PWR1" H 1950 1030 20  0001 C CNN
 F 1 "+5VA" H 1950 1000 30  0000 C CNN
 	1    1950 900
@@
 $EndComp
 $Comp
-L PWR_FLAG #FLG03
+L PWR_FLAG #FLG2
 U 1 1 51A0AF7D
 P 2600 4100
-F 0 "#FLG03" H 2600 4195 30  0001 C CNN
+F 0 "#FLG2" H 2600 4195 30  0001 C CNN
 F 1 "PWR_FLAG" H 2600 4280 30  0000 C CNN
 	1    2600 4100
@@
 $EndComp
 $Comp
-L PWR_FLAG #FLG04
+L PWR_FLAG #FLG1
 U 1 1 51A0AF32
 P 2150 1600
-F 0 "#FLG04" H 2150 1695 30  0001 C CNN
+F 0 "#FLG1" H 2150 1695 30  0001 C CNN
 F 1 "PWR_FLAG" H 2150 1780 30  0000 C CNN
 	1    2150 1600
@@
 $EndComp
 $Comp
-L +5VA #PWR05
+L +5VA #PWR2
 U 1 1 51A0AEED
 P 2400 1500
-F 0 "#PWR05" H 2400 1630 20  0001 C CNN
+F 0 "#PWR2" H 2400 1630 20  0001 C CNN
 F 1 "+5VA" H 2400 1600 30  0000 C CNN
 	1    2400 1500
@@
 $EndComp
 $Comp
-L AGND #PWR06
+L AGND #PWR3
 U 1 1 51A0AD37
 P 2900 4200
-F 0 "#PWR06" H 2900 4200 40  0001 C CNN
+F 0 "#PWR3" H 2900 4200 40  0001 C CNN
 F 1 "AGND" H 2900 4130 50  0000 C CNN
 	1    2900 4200

Commit message: import footprints
Parts:
- P35: footprint (none) -> PIN_ARRAY_5x2
Changed lines of the file:
@@
-EESchema Schematic File Version 2  date Sat 06 Jul 2013 02:58:34 PM CEST
+EESchema Schematic File Version 2  date Sat 03 Aug 2013 02:02:22 PM CEST
 LIBS:power
 LIBS:device
@@
 F 0 "P35" H 7800 5800 60  0000 C CNN
 F 1 "CONN_5X2" V 7800 5500 50  0000 C CNN
+F 2 "PIN_ARRAY_5x2" V 7900 5500 50  0001 C CNN
 	1    7800 5500
 	1    0    0    -1
@@
 NoConn ~ 7400 5600
 $Comp
-L AGND #PWR4
+L AGND #PWR01
 U 1 1 51B368C7
 P 3600 1350
-F 0 "#PWR4" H 3600 1350 40  0001 C CNN
+F 0 "#PWR01" H 3600 1350 40  0001 C CNN
 F 1 "AGND" H 3600 1280 50  0000 C CNN
 	1    3600 1350
@@
 	3600 1350 3600 1150
 $Comp
-L +5VA #PWR1
+L +5VA #PWR02
 U 1 1 51B368B6
 P 1950 900
-F 0 "#PWR1" H 1950 1030 20  0001 C CNN
+F 0 "#PWR02" H 1950 1030 20  0001 C CNN
 F 1 "+5VA" H 1950 1000 30  0000 C CNN
 	1    1950 900
@@
 $EndComp
 $Comp
-L PWR_FLAG #FLG2
+L PWR_FLAG #FLG03
 U 1 1 51A0AF7D
 P 2600 4100
-F 0 "#FLG2" H 2600 4195 30  0001 C CNN
+F 0 "#FLG03" H 2600 4195 30  0001 C CNN
 F 1 "PWR_FLAG" H 2600 4280 30  0000 C CNN
 	1    2600 4100
@@
 $EndComp
 $Comp
-L PWR_FLAG #FLG1
+L PWR_FLAG #FLG04
 U 1 1 51A0AF32
 P 2150 1600
-F 0 "#FLG1" H 2150 1695 30  0001 C CNN
+F 0 "#FLG04" H 2150 1695 30  0001 C CNN
 F 1 "PWR_FLAG" H 2150 1780 30  0000 C CNN
 	1    2150 1600
@@
 $EndComp
 $Comp
-L +5VA #PWR2
+L +5VA #PWR05
 U 1 1 51A0AEED
 P 2400 1500
-F 0 "#PWR2" H 2400 1630 20  0001 C CNN
+F 0 "#PWR05" H 2400 1630 20  0001 C CNN
 F 1 "+5VA" H 2400 1600 30  0000 C CNN
 	1    2400 1500
@@
 $EndComp
 $Comp
-L AGND #PWR3
+L AGND #PWR06
 U 1 1 51A0AD37
 P 2900 4200
-F 0 "#PWR3" H 2900 4200 40  0001 C CNN
+F 0 "#PWR06" H 2900 4200 40  0001 C CNN
 F 1 "AGND" H 2900 4130 50  0000 C CNN
 	1    2900 4200
