File: kicad-files/rev1/patch-shield-analog.sch (KiCad schematic (older format))
At the start: 38 parts, among them P1 CONN_1, P10 CONN_1, P11 CONN_1, P12 CONN_1, P13 CONN_1, P14 CONN_1, P15 CONN_1, P16 CONN_1, P17 CONN_1, P18 CONN_20X2, P19 CONN_1, P2 CONN_1, P20 CONN_1, P21 CONN_1, P22 CONN_1, P23 CONN_1, P24 CONN_1, P25 CONN_1, P26 CONN_1, P27 CONN_1, P28 CONN_1, P29 CONN_1, P3 CONN_1, P30 CONN_1, P31 CONN_1, P32 CONN_1, P33 CONN_1, P34 CONN_1, P35 CONN_5X2, P36 ARDUINO_SHIELD, P4 CONN_1, P5 CONN_1, P6 CONN_1, P7 CONN_1, P8 CONN_1, P9 CONN_1

Commit message: Another step in KiCAD 5 update
Co-authored-by: Ace Medlock <ace.medlock@gmail.com>
Co-authored-by: Eric Herman <eric@freesa.org>
Parts:
- D1: symbol patch-shield-analog-rescue:LED-RESCUE-patch-shield-analog -> patch-shield-analog-rescue:LED-RESCUE-patch-shield-analog-patch-shield-analog-rescue
- P1, P10, P11, P12, P13, P14, P15, P16, P17, P19, P2, P20, P21, P22, P23, P24, P25, P26, P27, P28, P29, P3, P30, P31, P32, P33, P34, P4, P5, P6, P7, P8, P9: symbol patch-shield-analog-rescue:CONN_1 -> patch-shield-analog-rescue:CONN_1-patch-shield-analog-rescue
- P18: symbol patch-shield-analog-rescue:CONN_20X2 -> patch-shield-analog-rescue:CONN_20X2-patch-shield-analog-rescue
- P35: symbol patch-shield-analog-rescue:CONN_5X2 -> patch-shield-analog-rescue:CONN_5X2-patch-shield-analog-rescue
- R1: symbol patch-shield-analog-rescue:R-RESCUE-patch-shield-analog -> patch-shield-analog-rescue:R-RESCUE-patch-shield-analog-patch-shield-analog-rescue
Changed lines of the file:
@@
 Connection ~ 6250 2600
 $Comp
-L patch-shield-analog-rescue:DGND #PWR01
+L patch-shield-analog-rescue:DGND-patch-shield-analog-rescue #PWR01
 U 1 1 5201A76F
 P 8750 4200
@@
 $EndComp
 $Comp
-L patch-shield-analog-rescue:DGND #PWR02
+L patch-shield-analog-rescue:DGND-patch-shield-analog-rescue #PWR02
 U 1 1 5201A769
 P 6250 2700
@@
 $EndComp
 $Comp
-L patch-shield-analog-rescue:DGND #PWR03
+L patch-shield-analog-rescue:DGND-patch-shield-analog-rescue #PWR03
 U 1 1 5201A761
 P 9150 1950
@@
 NoConn ~ 7400 5700
 $Comp
-L patch-shield-analog-rescue:CONN_5X2 P35
+L patch-shield-analog-rescue:CONN_5X2-patch-shield-analog-rescue P35
 U 1 1 51D81450
 P 7800 5500
@@
 NoConn ~ 7400 5600
 $Comp
-L patch-shield-analog-rescue:AGND #PWR04
+L patch-shield-analog-rescue:AGND-patch-shield-analog-rescue #PWR04
 U 1 1 51B368C7
 P 3600 1350
@@
 Power Indicator
 $Comp
-L patch-shield-analog-rescue:R-RESCUE-patch-shield-analog R1
+L patch-shield-analog-rescue:R-RESCUE-patch-shield-analog-patch-shield-analog-rescue R1
 U 1 1 51A0E0BF
 P 2400 1150
@@
 $EndComp
 $Comp
-L patch-shield-analog-rescue:LED-RESCUE-patch-shield-analog D1
+L patch-shield-analog-rescue:LED-RESCUE-patch-shield-analog-patch-shield-analog-rescue D1
 U 1 1 51A0E0BE
 P 3150 1150
@@
 $EndComp
 $Comp
-L patch-shield-analog-rescue:CONN_1 P2
+L patch-shield-analog-rescue:CONN_1-patch-shield-analog-rescue P2
 U 1 1 51A0B540
 P 1200 1950
@@
 $EndComp
 $Comp
-L patch-shield-analog-rescue:CONN_1 P3
+L patch-shield-analog-rescue:CONN_1-patch-shield-analog-rescue P3
 U 1 1 51A0B53F
 P 1200 2150
@@
 $EndComp
 $Comp
-L patch-shield-analog-rescue:CONN_1 P5
+L patch-shield-analog-rescue:CONN_1-patch-shield-analog-rescue P5
 U 1 1 51A0B53E
 P 1200 2550
@@
 $EndComp
 $Comp
-L patch-shield-analog-rescue:CONN_1 P4
+L patch-shield-analog-rescue:CONN_1-patch-shield-analog-rescue P4
 U 1 1 51A0B53D
 P 1200 2350
@@
 $EndComp
 $Comp
-L patch-shield-analog-rescue:CONN_1 P8
+L patch-shield-analog-rescue:CONN_1-patch-shield-analog-rescue P8
 U 1 1 51A0B53C
 P 1200 3150
@@
 $EndComp
 $Comp
-L patch-shield-analog-rescue:CONN_1 P9
+L patch-shield-analog-rescue:CONN_1-patch-shield-analog-rescue P9
 U 1 1 51A0B53B
 P 1200 3350
@@
 $EndComp
 $Comp
-L patch-shield-analog-rescue:CONN_1 P7
+L patch-shield-analog-rescue:CONN_1-patch-shield-analog-rescue P7
 U 1 1 51A0B53A
 P 1200 2950
@@
 $EndComp
 $Comp
-L patch-shield-analog-rescue:CONN_1 P6
+L patch-shield-analog-rescue:CONN_1-patch-shield-analog-rescue P6
 U 1 1 51A0B539
 P 1200 2750
@@
 $EndComp
 $Comp
-L patch-shield-analog-rescue:CONN_1 P31
+L patch-shield-analog-rescue:CONN_1-patch-shield-analog-rescue P31
 U 1 1 51A0B512
 P 4600 2750
@@
 $EndComp
 $Comp
-L patch-shield-analog-rescue:CONN_1 P32
+L patch-shield-analog-rescue:CONN_1-patch-shield-analog-rescue P32
 U 1 1 51A0B511
 P 4600 2950
@@
 $EndComp
 $Comp
-L patch-shield-analog-rescue:CONN_1 P34
+L patch-shield-analog-rescue:CONN_1-patch-shield-analog-rescue P34
 U 1 1 51A0B510
 P 4600 3350
@@
 $EndComp
 $Comp
-L patch-shield-analog-rescue:CONN_1 P33
+L patch-shield-analog-rescue:CONN_1-patch-shield-analog-rescue P33
 U 1 1 51A0B50F
 P 4600 3150
@@
 $EndComp
 $Comp
-L patch-shield-analog-rescue:CONN_1 P29
+L patch-shield-analog-rescue:CONN_1-patch-shield-analog-rescue P29
 U 1 1 51A0B508
 P 4600 2350
@@
 $EndComp
 $Comp
-L patch-shield-analog-rescue:CONN_1 P30
+L patch-shield-analog-rescue:CONN_1-patch-shield-analog-rescue P30
 U 1 1 51A0B507
 P 4600 2550
@@
 $EndComp
 $Comp
-L patch-shield-analog-rescue:CONN_1 P28
+L patch-shield-analog-rescue:CONN_1-patch-shield-analog-rescue P28
 U 1 1 51A0B4FC
 P 4600 2150
@@
 $EndComp
 $Comp
-L patch-shield-analog-rescue:CONN_1 P27
+L patch-shield-analog-rescue:CONN_1-patch-shield-analog-rescue P27
 U 1 1 51A0B4B7
 P 4600 1950
@@
 BIASOUT
 $Comp
-L patch-shield-analog-rescue:CONN_1 P1
+L patch-shield-analog-rescue:CONN_1-patch-shield-analog-rescue P1
 U 1 1 51A0AFA6
 P 850 3550
@@
 $EndComp
 $Comp
-L patch-shield-analog-rescue:CONN_1 P10
+L patch-shield-analog-rescue:CONN_1-patch-shield-analog-rescue P10
 U 1 1 51A0ADBD
 P 1600 1950
@@
 $EndComp
 $Comp
-L patch-shield-analog-rescue:CONN_1 P11
+L patch-shield-analog-rescue:CONN_1-patch-shield-analog-rescue P11
 U 1 1 51A0ADBC
 P 1600 2150
@@
 $EndComp
 $Comp
-L patch-shield-analog-rescue:CONN_1 P13
+L patch-shield-analog-rescue:CONN_1-patch-shield-analog-rescue P13
 U 1 1 51A0ADBB
 P 1600 2550
@@
 $EndComp
 $Comp
-L patch-shield-analog-rescue:CONN_1 P12
+L patch-shield-analog-rescue:CONN_1-patch-shield-analog-rescue P12
 U 1 1 51A0ADBA
 P 1600 2350
@@
 $EndComp
 $Comp
-L patch-shield-analog-rescue:CONN_1 P16
+L patch-shield-analog-rescue:CONN_1-patch-shield-analog-rescue P16
 U 1 1 51A0ADB9
 P 1600 3150
@@
 $EndComp
 $Comp
-L patch-shield-analog-rescue:CONN_1 P17
+L patch-shield-analog-rescue:CONN_1-patch-shield-analog-rescue P17
 U 1 1 51A0ADB8
 P 1600 3350
@@
 $EndComp
 $Comp
-L patch-shield-analog-rescue:CONN_1 P15
+L patch-shield-analog-rescue:CONN_1-patch-shield-analog-rescue P15
 U 1 1 51A0ADB7
 P 1600 2950
@@
 $EndComp
 $Comp
-L patch-shield-analog-rescue:CONN_1 P14
+L patch-shield-analog-rescue:CONN_1-patch-shield-analog-rescue P14
 U 1 1 51A0ADB6
 P 1600 2750
@@
 $EndComp
 $Comp
-L patch-shield-analog-rescue:AGND #PWR09
+L patch-shield-analog-rescue:AGND-patch-shield-analog-rescue #PWR09
 U 1 1 51A0AD37
 P 2900 4200
@@
 $EndComp
 $Comp
-L patch-shield-analog-rescue:CONN_1 P23
+L patch-shield-analog-rescue:CONN_1-patch-shield-analog-rescue P23
 U 1 1 51A0AC59
 P 4200 2750
@@
 $EndComp
 $Comp
-L patch-shield-analog-rescue:CONN_1 P24
+L patch-shield-analog-rescue:CONN_1-patch-shield-analog-rescue P24
 U 1 1 51A0AC58
 P 4200 2950
@@
 $EndComp
 $Comp
-L patch-shield-analog-rescue:CONN_1 P26
+L patch-shield-analog-rescue:CONN_1-patch-shield-analog-rescue P26
 U 1 1 51A0AC57
 P 4200 3350
@@
 $EndComp
 $Comp
-L patch-shield-analog-rescue:CONN_1 P25
+L patch-shield-analog-rescue:CONN_1-patch-shield-analog-rescue P25
 U 1 1 51A0AC56
 P 4200 3150
@@
 $EndComp
 $Comp
-L patch-shield-analog-rescue:CONN_1 P21
+L patch-shield-analog-rescue:CONN_1-patch-shield-analog-rescue P21
 U 1 1 51A0AC3D
 P 4200 2350
@@
 $EndComp
 $Comp
-L patch-shield-analog-rescue:CONN_1 P22
+L patch-shield-analog-rescue:CONN_1-patch-shield-analog-rescue P22
 U 1 1 51A0AC3C
 P 4200 2550
@@
 $EndComp
 $Comp
-L patch-shield-analog-rescue:CONN_1 P20
+L patch-shield-analog-rescue:CONN_1-patch-shield-analog-rescue P20
 U 1 1 51A0AC26
 P 4200 2150
@@
 $EndComp
 $Comp
-L patch-shield-analog-rescue:CONN_1 P19
+L patch-shield-analog-rescue:CONN_1-patch-shield-analog-rescue P19
 U 1 1 51A0ABA4
 P 4200 1950
@@
 $EndComp
 $Comp
-L patch-shield-analog-rescue:CONN_20X2 P18
+L patch-shield-analog-rescue:CONN_20X2-patch-shield-analog-rescue P18
 U 1 1 51A0A305
 P 2900 2700
