File: kicad-files/rev1/bnc-shield.sch (KiCad schematic (older format))
At the start: 128 parts, among them P1 BNC, P10 CONN_20X2, P11 CONN_4, P12 CONN_4X2, P13 ARDUINO_SHIELD, P2 BNC, P3 BNC, P4 BNC, P5 BNC, P6 BNC, P7 BNC, P8 BNC, P9 CONN_1, U1 TS5A4624, U10 TS5A4624, U11 TS5A4624, U12 TS5A4624, U13 TS5A4624, U14 TS5A4624, U15 TS5A4624, U16 TS5A4624, U17 TS5A4624, U18 74HC595, U19 74HC595, U2 TS5A4624, U20 SI8661, U21 74HC595, U22 74HC595, U23 CAT24C128, U3 TS5A4624, U4 TS5A4624, U5 TS5A4624, U6 TS5A4624, U7 TS5A4624, U8 TS5A4624, U9 TPS7A49XX

Commit message: remove unused DAISY_SERIAL_4
Connections:
- net labels removed: LED_SERIAL_DAISY_4, LED_SERIAL_DAISY_4_ISO
- wire segments 560 -> 558
- no-connect marks 17 -> 19

Commit message: merge GPIO and Supplemental IO connectors
Parts:
- removed L5: INDUCTOR, symbol INDUCTOR
- removed P11: CONN_4, symbol CONN_4
- removed P12: CONN_4X2, symbol CONN_4X2
- added P?: CONN_5X2, symbol CONN_5X2
Connections:
- wire segments 558 -> 553
Other:
- note added: "Supplemental digital IO header"
Changed lines of the file:
@@
-EESchema Schematic File Version 2  date Sat 22 Jun 2013 02:09:31 PM CEST
+EESchema Schematic File Version 2  date Sat 06 Jul 2013 02:56:58 PM CEST
 LIBS:power
 LIBS:device
@@
 Sheet 1 1
 Title "noname.sch"
-Date "22 jun 2013"
+Date "6 jul 2013"
 Rev ""
 Comp ""
@@
 Comment4 ""
 $EndDescr
+Text Label 21700 5050 2    60   ~ 0
+LED_SERIAL
+Text Label 21700 4950 2    60   ~ 0
+LED_SHIFT_REG_CLK
+Text Label 21700 4850 2    60   ~ 0
+LED_SHIFT_REG_CLEAR
+Text Label 17600 5050 0    60   ~ 0
+ADS129x_GPIO4
+Text Label 17600 4950 0    60   ~ 0
+ADS129x_GPIO3
+Text Label 17600 4850 0    60   ~ 0
+ADS129x_GPIO2
+Text Label 17600 4750 0    60   ~ 0
+ADS129x_GPIO1
+Text Label 21700 4650 2    60   ~ 0
+LED_LATCH_CLK
+Text Label 21700 4750 2    60   ~ 0
+LED_OUTPUT_ENABLE_INPUT
+Text Notes 18950 4100 0    60   ~ 0
+Supplemental digital IO header
+$Comp
+L CONN_5X2 P?
+U 1 1 51D8130B
+P 19650 4850
+F 0 "P?" H 19650 5150 60  0000 C CNN
+F 1 "CONN_5X2" V 19650 4850 50  0000 C CNN
+	1    19650 4850
+	1    0    0    -1
+$EndComp
+Wire Wire Line
+	19250 4750 17600 4750
+Wire Wire Line
+	19250 4850 17600 4850
+Wire Wire Line
+	17600 4950 19250 4950
+Wire Wire Line
+	17600 5050 19250 5050
+Wire Wire Line
+	21700 4950 20050 4950
+Wire Wire Line
+	21700 5050 20050 5050
+Wire Wire Line
+	21700 4650 20050 4650
+Wire Wire Line
+	21700 4750 20050 4750
+Wire Wire Line
+	21700 4850 20050 4850
 Connection ~ 11000 2550
 Wire Wire Line
@@
 Wire Wire Line
 	11000 2450 11100 2450
-Connection ~ 20100 4700
-Wire Wire Line
-	20050 4700 20100 4700
 Wire Notes Line
 	11650 1600 11650 550
@@
 Wire Wire Line
 	18700 3650 18150 3650
-Wire Wire Line
-	14850 1950 16450 1950
-Wire Wire Line
-	14850 1850 16450 1850
-Wire Wire Line
-	14850 1750 16450 1750
-Wire Wire Line
-	14850 1650 16450 1650
-Wire Wire Line
-	21700 4400 20050 4400
-Wire Wire Line
-	19250 4600 17600 4600
-Wire Wire Line
-	19250 4500 17600 4500
-Wire Wire Line
-	19250 4700 17600 4700
-Wire Wire Line
-	21700 4500 20050 4500
-Connection ~ 18350 4400
-Wire Wire Line
-	18350 4350 18350 4400
-Wire Wire Line
-	19100 4400 19250 4400
-Wire Wire Line
-	18500 4400 18000 4400
-Wire Wire Line
-	18000 4400 18000 4300
+Connection ~ 18950 4650
+Wire Wire Line
+	18950 4600 18950 4650
+Wire Wire Line
+	19100 4650 19250 4650
+Wire Wire Line
+	19100 4650 18600 4650
+Wire Wire Line
+	18600 4650 18600 4550
 Connection ~ 4950 3300
 Wire Wire Line
@@
 Wire Notes Line
 	11650 2800 11650 16050
-Wire Wire Line
-	20050 4600 20100 4600
-Wire Wire Line
-	20100 4600 20100 5100
-Wire Wire Line
-	20300 5000 20300 5050
-Wire Wire Line
-	20300 5050 20100 5050
-Connection ~ 20100 5050
 Connection ~ 18200 12950
 Wire Wire Line
@@
 F 1 "CAT24C128" H 18400 13200 60  0000 C CNN
 	1    18200 13550
-	1    0    0    -1
-$EndComp
-$Comp
-L CONN_4X2 P12
-U 1 1 51C5882E
-P 19650 4550
-F 0 "P12" H 19650 4800 50  0000 C CNN
-F 1 "CONN_4X2" V 19650 4550 40  0000 C CNN
-	1    19650 4550
 	1    0    0    -1
 $EndComp
@@
 	1    0    0    -1
 $EndComp
-Text Label 14850 1650 0    60   ~ 0
-ADS129x_GPIO1
-Text Label 14850 1750 0    60   ~ 0
-ADS129x_GPIO2
-Text Label 14850 1850 0    60   ~ 0
-ADS129x_GPIO3
-Text Label 14850 1950 0    60   ~ 0
-ADS129x_GPIO4
-$Comp
-L CONN_4 P11
-U 1 1 51B42FDF
-P 16800 1800
-F 0 "P11" V 16750 1800 50  0000 C CNN
-F 1 "CONN_4" V 16850 1800 50  0000 C CNN
-	1    16800 1800
-	1    0    0    -1
-$EndComp
 $Comp
 L +3.3V #PWR71
 U 1 1 51B42CF8
-P 18000 4300
-F 0 "#PWR71" H 18000 4260 30  0001 C CNN
-F 1 "+3.3V" H 18000 4410 30  0000 C CNN
-	1    18000 4300
+P 18600 4550
+F 0 "#PWR71" H 18600 4510 30  0001 C CNN
+F 1 "+3.3V" H 18600 4660 30  0000 C CNN
+	1    18600 4550
 	1    0    0    -1
 $EndComp
@@
 L PWR_FLAG #FLG7
 U 1 1 51B42CF7
-P 18350 4350
-F 0 "#FLG7" H 18350 4445 30  0001 C CNN
-F 1 "PWR_FLAG" H 18350 4530 30  0000 C CNN
-	1    18350 4350
-	1    0    0    -1
-$EndComp
-$Comp
-L INDUCTOR L5
-U 1 1 51B42CF6
-P 18800 4400
-F 0 "L5" V 18750 4400 40  0000 C CNN
-F 1 "INDUCTOR" V 18900 4400 40  0000 C CNN
-	1    18800 4400
-	0    -1   -1   0
-$EndComp
-Text Label 21700 4500 2    60   ~ 0
-LED_OUTPUT_ENABLE_INPUT
-Text Label 21700 4400 2    60   ~ 0
-LED_LATCH_CLK
-$Comp
-L GND #PWR81
-U 1 1 51B42CF4
-P 20100 5100
-F 0 "#PWR81" H 20100 5100 30  0001 C CNN
-F 1 "GND" H 20100 5030 30  0001 C CNN
-	1    20100 5100
-	1    0    0    -1
-$EndComp
-Text Label 17600 4700 0    60   ~ 0
-LED_SHIFT_REG_CLEAR
-Text Label 17600 4600 0    60   ~ 0
-LED_SHIFT_REG_CLK
-Text Label 17600 4500 0    60   ~ 0
-LED_SERIAL
-$Comp
-L PWR_FLAG #FLG9
-U 1 1 51B42CF3
-P 20300 5000
-F 0 "#FLG9" H 20300 5095 30  0001 C CNN
-F 1 "PWR_FLAG" H 20300 5180 30  0000 C CNN
-	1    20300 5000
-	1    0    0    -1
-$EndComp
+P 18950 4600
+F 0 "#FLG7" H 18950 4695 30  0001 C CNN
+F 1 "PWR_FLAG" H 18950 4780 30  0000 C CNN
+	1    18950 4600
+	1    0    0    -1
+$EndComp

Commit message: add bnc connectors for digital signals
Parts:
- added P? (x8): BNC, symbol BNC
Connections:
- wire segments 553 -> 568

Commit message: add voltage translator for digital BNC connectors, fix some ERC errors
Parts:
- added U24: TXS0108E, symbol TXS0108E
- gave numbers to parts that had none: 9
Connections:
- wire segments 568 -> 606
- no-connect marks 19 -> 41
Other:
- note added: "3.3V CMOS"
- note added: "5V TTL/CMOS"
- note added: "5V to 3.3V bidirectional\nvoltage translator"

Commit message: remove implicit connection across isolation from 74HC595
Parts:
- removed U18, U19, U21, U22: 74HC595, symbol 74HC595
- added U18, U19, U21, U22: 74HC595, symbol 74HC595_VIS
Connections:
- wire segments 606 -> 607
- no-connect marks 41 -> 40

Commit message: assigned footprints for bnc shield
Parts:
- C1, C12, C13, C14, C15, C16, C17, C18, C19, C2, C21, C22, C25, C28, C3, C31, C32, C33, C4, C5, C6, C7, C8, R1, R11, R15, R16, R17, R18, R19, R2, R21, R23, R25, R27, R28, R29, R3, R30, R31, R32, R33, R34, R35, R4, R5, R7, R9: footprint (none) -> SM0603
- C20, C9: footprint SM1210 -> SM0805
- C23, C24, C26, C27, C29, C30, C34, L1, L2, L3, L4, L6, R10, R12, R20, R22, R24, R26, R6, R8: footprint (none) -> SM0805
- D1, D10, D11, D12, D13, D14, D15, D16, D17, D2, D3, D4, D5, D6, D7, D8, D9: footprint (none) -> LED-0603
- P1, P11, P12, P14, P15, P16, P17, P18, P19, P2, P3, P4, P5, P6, P7, P8: footprint (none) -> BNC-6x89mm
- P10: footprint (none) -> PIN_ARRAY_20X2
- P13: footprint (none) -> arduino_shield
- P20: footprint (none) -> PIN_ARRAY_5x2
- P9: footprint (none) -> banana-jack
- U1, U10, U11, U12, U13, U14, U15, U16, U17, U2, U3, U4, U5, U6, U7, U8: footprint (none) -> SC70-6
- U18, U19, U21, U22: footprint (none) -> TSSOP16
- U20: footprint (none) -> SO16W
- U23: footprint (none) -> SO8E
- U24: footprint (none) -> TSSOP20

Commit message: add pull-down resistor for Output Enable on BNC board
Parts:
- added R36: 10k, symbol R
Connections:
- wire segments 607 -> 609

Commit message: add digital status and activity LEDs to BNC board
Parts:
- added C35, C36: 10uF, SM0805, symbol C
- added C37, C38: 100nF, SM0603, symbol C
- added D18, D19, D20, D21, D22, D23, D24, D25, D26, D27, D28, D29, D30, D31, D32, D33, D34, D35, D36, D37, D38, D39, D40, D41: LED, LED-0603, symbol LED
- added R37, R38, R39, R40, R41, R42, R43, R44, R45, R46, R47, R48, R49, R50, R51, R52: 560, SM0603, symbol R
- added U25, U26: 74HC595, TSSOP16, symbol 74HC595_VIS
Connections:
- net labels added: GREEN_IN_D1, GREEN_IN_D2, GREEN_IN_D3, GREEN_IN_D4, GREEN_IN_D5, GREEN_IN_D6, GREEN_IN_D7, GREEN_IN_D8, GREEN_OUT_D1, GREEN_OUT_D2, GREEN_OUT_D3, GREEN_OUT_D4, GREEN_OUT_D5, GREEN_OUT_D6, GREEN_OUT_D7, GREEN_OUT_D8, LED_SERIAL_DAISY_4, LED_SERIAL_DAISY_4_ISO
- net labels removed: LED_SERIAL_DAISY_2, LED_SERIAL_DAISY_2_ISO
- wire segments 609 -> 733
Other:
- note added: "Analog Input Status LEDS"
- note added: "Digital I/O Activity LEDs"
- note added: "Digital I/O Status LEDs"
- moved on the sheet: C29, C30, C31, C32, C33, C34, D1, D10, D11, D12, D13, D14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
