File: kicad-files/rev1/patch-shield-digital.sch (KiCad schematic (older format))
At the start: 68 parts, among them P1 CONN_5X2, P2 ARDUINO_SHIELD, U1 CAT24C128, U5 74HC595, U6 74HC595, U7 74HC595, U8 74HC595

Commit message: make Rules Check pass
Connections:
- wire segments 250 -> 252
- no-connect marks 32 -> 34
Changed lines of the file:
@@
-EESchema Schematic File Version 2  date Sat 06 Jul 2013 03:03:50 PM CEST
+EESchema Schematic File Version 2  date Sat 03 Aug 2013 02:16:51 PM CEST
 LIBS:power
 LIBS:device
@@
 Sheet 1 1
 Title "noname.sch"
-Date "6 jul 2013"
+Date "3 aug 2013"
 Rev ""
 Comp ""
@@
 Comment4 ""
 $EndDescr
+Text Label 20000 3900 2    60   ~ 0
+PA17_SDA1
+Text Label 20000 3800 2    60   ~ 0
+PA18_SCL1
+Wire Wire Line
+	20000 3800 19300 3800
+Wire Wire Line
+	19300 3900 20000 3900
+NoConn ~ 15950 7950
+NoConn ~ 15950 7850
+NoConn ~ 15950 7750
+NoConn ~ 15950 7650
 Connection ~ 16450 4900
 Wire Wire Line
-	16450 4900 16000 4900
+	16000 4900 16450 4900
 Wire Wire Line
 	16000 4900 16000 4700
@@
 Connection ~ 17500 10800
 Wire Wire Line
-	17500 10800 16700 10800
+	16700 10800 17500 10800
 Wire Wire Line
 	16700 10800 16700 11200
@@
 Connection ~ 18400 12000
 Wire Wire Line
-	18400 12100 18400 12000
+	18400 12000 18400 12100
 Wire Wire Line
 	16700 12000 18800 12000
@@
 	16700 11300 16800 11300
 Wire Wire Line
-	18400 9800 17500 9800
+	17500 9800 18400 9800
 Wire Wire Line
 	17900 10300 17900 10500
@@
 	17500 12000 17500 11900
 Wire Wire Line
-	17500 9800 17500 10900
+	17500 10900 17500 9800
 Wire Wire Line
 	19300 4100 19500 4100
@@
 	16450 4700 16700 4700
 Wire Wire Line
-	16700 4500 16450 4500
-Wire Wire Line
-	16450 4500 16450 4100
+	16450 4500 16700 4500
+Wire Wire Line
+	16450 4100 16450 4500
 Wire Wire Line
 	16700 4300 16450 4300
@@
 	10050 8850 10150 8850
 Wire Wire Line
-	11150 1350 10750 1350
+	10750 1350 11150 1350
 Wire Wire Line
 	10750 1350 10750 1300
 Connection ~ 10550 850
 Wire Wire Line
-	11150 900  11150 850
+	11150 850  11150 900
 Wire Wire Line
 	11150 850  10550 850
@@
 Connection ~ 5400 2650
 Wire Wire Line
-	5400 2650 5400 2350
+	5400 2350 5400 2650
 Wire Wire Line
 	5400 2350 5250 2350
@@
 	4850 1250 4100 1250
 Wire Wire Line
-	6050 1250 6600 1250
+	6600 1250 6050 1250
 Wire Wire Line
 	5250 1250 5550 1250
@@
 Connection ~ 5400 1950
 Wire Wire Line
-	5400 1950 5400 1650
+	5400 1650 5400 1950
 Wire Wire Line
 	5400 1650 5250 1650
@@
 Connection ~ 5400 4050
 Wire Wire Line
-	5400 4050 5400 3750
+	5400 3750 5400 4050
 Wire Wire Line
 	5400 3750 5250 3750
@@
 Connection ~ 5400 6150
 Wire Wire Line
-	5400 6150 5400 5850
+	5400 5850 5400 6150
 Wire Wire Line
 	5400 5850 5250 5850
@@
 Connection ~ 6600 1950
 Wire Wire Line
-	6600 1250 6600 6650
+	6600 6650 6600 1250
 Connection ~ 6600 6150
 Connection ~ 750  6200
@@
 Connection ~ 1950 5500
 Wire Wire Line
-	1950 5500 1950 5200
+	1950 5200 1950 5500
 Wire Wire Line
 	1950 5200 2100 5200
@@
 Connection ~ 1950 4800
 Wire Wire Line
-	1950 4800 1950 4500
+	1950 4500 1950 4800
 Wire Wire Line
 	1950 4500 2100 4500
@@
 Connection ~ 1950 1300
 Wire Wire Line
-	1950 1300 1950 1000
+	1950 1000 1950 1300
 Wire Wire Line
 	1950 1000 2100 1000
@@
 Connection ~ 1950 3400
 Wire Wire Line
-	1950 3400 1950 3100
+	1950 3100 1950 3400
 Wire Wire Line
 	1950 3100 2100 3100
@@
 	10750 3750 11150 3750
 Wire Wire Line
-	11150 6150 10750 6150
+	10750 6150 11150 6150
 Wire Wire Line
 	10750 6150 10750 6100
 Connection ~ 10550 5650
 Wire Wire Line
-	11150 5700 11150 5650
+	11150 5650 11150 5700
 Wire Wire Line
 	11150 5650 10550 5650
@@
 NoConn ~ 19300 4200
 NoConn ~ 19300 4000
-NoConn ~ 19300 3900
-NoConn ~ 19300 3800
 $Comp
 L GND #PWR06
@@
 	0    1    1    0
 $EndComp
-Text Label 4600 3350 2    60   ~ 0
+Text Label 4100 3350 0    60   ~ 0
 YELLOW_5P
-Text Label 4556 3050 2    60   ~ 0
+Text Label 4100 3050 0    60   ~ 0
 GREEN_5P
-Text Label 4556 2350 2    60   ~ 0
+Text Label 4100 2350 0    60   ~ 0
 GREEN_6P
-Text Label 4600 2650 2    60   ~ 0
+Text Label 4100 2650 0    60   ~ 0
 YELLOW_6P
 $Comp
@@
 	0    1    1    0
 $EndComp
-Text Label 4600 1250 2    60   ~ 0
+Text Label 4100 1250 0    60   ~ 0
 YELLOW_8P
-Text Label 4556 950  2    60   ~ 0
+Text Label 4100 950  0    60   ~ 0
 GREEN_8P
-Text Label 4556 1650 2    60   ~ 0
+Text Label 4100 1650 0    60   ~ 0
 GREEN_7P
-Text Label 4600 1950 2    60   ~ 0
+Text Label 4100 1950 0    60   ~ 0
 YELLOW_7P
 $Comp
@@
 	0    1    1    0
 $EndComp
-Text Label 4600 4750 2    60   ~ 0
+Text Label 4100 4750 0    60   ~ 0
 YELLOW_3P
-Text Label 4556 4450 2    60   ~ 0
+Text Label 4100 4450 0    60   ~ 0
 GREEN_3P
-Text Label 4556 3750 2    60   ~ 0
+Text Label 4100 3750 0    60   ~ 0
 GREEN_4P
-Text Label 4600 4050 2    60   ~ 0
+Text Label 4100 4050 0    60   ~ 0
 YELLOW_4P
 $Comp
@@
 	0    1    1    0
 $EndComp
-Text Label 4600 5450 2    60   ~ 0
+Text Label 4100 5450 0    60   ~ 0
 YELLOW_2P
-Text Label 4556 5150 2    60   ~ 0
+Text Label 4100 5150 0    60   ~ 0
 GREEN_2P
-Text Label 4556 5850 2    60   ~ 0
+Text Label 4100 5850 0    60   ~ 0
 GREEN_1P
-Text Label 4600 6150 2    60   ~ 0
+Text Label 4100 6150 0    60   ~ 0
 YELLOW_1P
 $Comp

Commit message: add footprints to patch-shield-digital
Parts:
- C1, C10, C11, C12, C13, R1, R10, R11, R12, R13, R14, R15, R16, R17, R18, R2, R3, R4, R5, R6, R7, R8: footprint (none) -> SM0603
- C2, C6, C7, C8, C9, L1: footprint (none) -> SM0805
- D1, D10, D11, D12, D13, D14, D15, D16, D18, D19, D2, D20, D21, D22, D23, D24, D25, D26, D27, D28, D29, D3, D30, D31, D32, D33, D34, D4, D5, D6, D7, D8, D9: footprint (none) -> LED-0603
- P1: footprint (none) -> PIN_ARRAY_5x2
- P2: footprint (none) -> arduino_shield
- U1: footprint (none) -> SOIC8
- U5, U6, U7, U8: footprint (none) -> SO16E

Commit message: change serial-to-par footprint from SO16E to TSSOP16
Parts:
- U5, U6, U7, U8: footprint SO16E -> TSSOP16
Changed lines of the file:
@@
-EESchema Schematic File Version 2  date Sat 03 Aug 2013 02:19:31 PM CEST
+EESchema Schematic File Version 2  date Sat 03 Aug 2013 02:35:40 PM CEST
 LIBS:power
 LIBS:device
@@
 F 0 "U8" H 11000 9900 70  0000 C CNN
 F 1 "74HC595" H 10850 8700 70  0000 C CNN
-F 2 "SO16E" H 10850 8800 70  0001 C CNN
+F 2 "TSSOP16" H 10850 8800 70  0001 C CNN
 	1    10850 9300
 	1    0    0    -1
@@
 F 0 "U7" H 11000 7500 70  0000 C CNN
 F 1 "74HC595" H 10850 6300 70  0000 C CNN
-F 2 "SO16E" H 10850 6400 70  0001 C CNN
+F 2 "TSSOP16" H 10850 6400 70  0001 C CNN
 	1    10850 6900
 	1    0    0    -1
@@
 F 0 "U6" H 11000 5100 70  0000 C CNN
 F 1 "74HC595" H 10850 3900 70  0000 C CNN
-F 2 "SO16E" H 10850 4000 70  0001 C CNN
+F 2 "TSSOP16" H 10850 4000 70  0001 C CNN
 	1    10850 4500
 	1    0    0    -1
@@
 F 0 "U5" H 11000 2700 70  0000 C CNN
 F 1 "74HC595" H 10850 1500 70  0000 C CNN
-F 2 "SO16E" H 10850 1600 70  0001 C CNN
+F 2 "TSSOP16" H 10850 1600 70  0001 C CNN
 	1    10850 2100
 	1    0    0    -1

Commit message: add series resistors for shift registers for LEDs
Parts:
- added R19, R20, R21, R22, R23, R24, R25, R9: 47, SM0603, symbol R
Connections:
- wire segments 252 -> 260
